File: hardware/plush-toy-mainboard/plush-toy-mainboard.kicad_sch (KiCad schematic)
At the start: 110 parts, among them U1 ESP32-S3-WROOM-1-N16R8

Commit message: feat(pcb): complete plush toy mainboard routing
Parts:
- H1, H2, H3, H4, R_SIOC, R_SIOD, TP_3V3, TP_E0, TP_E1, TP_E10, TP_E11, TP_E2, TP_E3, TP_E4, TP_E5, TP_E6, TP_E7, TP_E8, TP_E9, TP_GATE, TP_GND, TP_OE, TP_PGND, TP_SCL, TP_SDA, TP_TX, TP_VBUS, TP_VMOT: now left out of the parts list

Commit message: fix(pcb): finalize plush toy preflight respin
Parts:
- removed TP_E0: TOUCH_E0, TestPoint:TestPoint_Pad_D1.0mm, symbol Connector:TestPoint
- added C_BUCK_HF, C_EFUSE_IN: 100nF, Capacitor_SMD:C_0402_1005Metric, symbol Device:C
- added C_EFUSE_DVDT: 3.3nF, Capacitor_SMD:C_0402_1005Metric, symbol Device:C
- added J_TOUCH: Head Touch, Connector_JST:JST_PH_B2B-PH-K_1x02_P2.00mm_Vertical, symbol Connector_Generic:Conn_01x02
- added R_EFUSE_ILM: 1.02k, Resistor_SMD:R_0402_1005Metric, symbol Device:R
- added U_EFUSE: TPS259531DSGR, Package_SON:Texas_DSG0008A_WSON-8-1EP_2x2mm_P0.5mm_EP0.9x1.6mm_ThermalVias, symbol plush:TPS259531
- D_LED: value WS2812B-2020 -> WS2812B-2020-V6; LCSC C965555 -> C52917434
- J_HEAT, J_LCD_L, J_LCD_R, J_NTC, J_SERVO_L, J_SERVO_R, J_SPK, J_VMOT: now left out of the parts list
- R_SIOC, R_SIOD: now fitted; now in the parts list
Connections:
- net GND: now also C_BUCK_HF.2, C_EFUSE_DVDT.2, C_EFUSE_IN.2, J_TOUCH.2 (Pin_2), R_EFUSE_ILM.2, U_EFUSE.8 (GND), U_EFUSE.9 (EP)
- net TOUCH_E0: now also J_TOUCH.1 (Pin_1)
- net VBUS: now also C_BUCK_HF.1, U_EFUSE.5 (OUT); no longer F_USB.2
- new net EFUSE_DVDT: C_EFUSE_DVDT.1, U_EFUSE.1 (dVdt)
- new net EFUSE_ILM: R_EFUSE_ILM.1, U_EFUSE.7 (ILM)
- new net VBUS_FUSED: C_EFUSE_IN.1, F_USB.2, U_EFUSE.2 (EN/UVLO), U_EFUSE.3 (IN), U_EFUSE.4 (IN)
- no-connect marks 48 -> 49
