File: hardware/plush-toy-mainboard/plush-toy-mainboard.kicad_sch (KiCad schematic)
At the start: 115 parts, among them U1 ESP32-S3-WROOM-1-N16R8

Commit message: feat(pcb): GPIO48 改驱动双眼背光，撤销板载 RGB 灯
屏幕换成带独立 BL 引脚的型号（7 针 → 8 针 RST/CS/DC/SDA/SCL/GND/VCC/BL）。
D_LED 与 C_LED 整体撤销，GPIO48 改作两眼共用的 25kHz 背光 PWM：眼睛本身已能
表达设备状态，换来统一亮度调节和休眠关背光。摄像头、音频、USB、SPI 与
strapping 脚均不受影响。

硬件：
- 新增 AO3401A 高边开关 Q_LCD_BL（与 Q_REV 同料号 C15127），栅极串 100Ω、
  上拉 100k 至 +3V3，保证 LEDC 配置前 GPIO48 浮空时背光默认灭。
- 开关放在双屏排针正下方的空区：LCD_BL 只需 4~11mm 就接到两排 8 脚，横穿
  板子的改成 25kHz 栅极信号。此处 x<62，In2.Cu 的 +3V3 覆铜仍在（覆铜止于
  x=62），源极和上拉能就近打孔取电。
- 新增 apply_backlight_eco.py：整板重新自动布线会在 U_TOUCH/J_CAM 密集区失去
  已收敛路径，因此只做局部 ECO，且 DRC/未连接/原理图一致性全过才覆盖正式 PCB。
- 排针加到 8 针后 8 脚右移 2.54mm，J_VMOT 旁两行 5V 警告标签离屏排针只剩
  5.5mm，又会被读成「屏幕座是 5V」——正是 2026-09-14 评审要消除的误读。右边
  顶着 H3 安装孔挪不动，故第二行去掉与第一行重复的「5V」，只留设计方案要求的
  「电机/加热专用」，两行右挪后间距 7.4mm。

固件：
- DISPLAY_BACKLIGHT_PIN=GPIO48 + DISPLAY_BACKLIGHT_OUTPUT_INVERT（低电平导通
  高边 P-MOS），改用 PwmBacklight；移除 GetLed 覆写，回落到基类 NoLed。

验证：DRC/未连接/原理图一致性只剩 2 条既有的 U1 丝印告警；113 项测试全过；
idf.py build 通过；fab 与渲染图已重出。

Co-Authored-By: Claude Opus 5 <noreply@anthropic.com>
Parts:
- removed C_LED: 100nF, Capacitor_SMD:C_0402_1005Metric, symbol Device:C
- removed D_LED: WS2812B-2020-V6, LED_SMD:LED_WS2812B-2020_PLCC4_2.0x2.0mm, symbol LED:WS2812B-2020
- added Q_LCD_BL: AO3401A, Package_TO_SOT_SMD:SOT-23, symbol Transistor_FET:AO3401A
- added R_LCD_BL_GATE: 100, Resistor_SMD:R_0402_1005Metric, symbol Device:R
- added R_LCD_BL_OFF: 100k, Resistor_SMD:R_0402_1005Metric, symbol Device:R
- J_LCD_L, J_LCD_R: footprint Connector_PinHeader_2.54mm:PinHeader_1x07_P2.54mm_Vertical -> Connector_PinHeader_2.54mm:PinHeader_1x08_P2.54mm_Vertical; symbol Connector_Generic:Conn_01x07 -> Connector_Generic:Conn_01x08
Connections:
- net +3V3: now also Q_LCD_BL.2 (S), R_LCD_BL_OFF.1
- net LED_RGB renamed LCD_BL_PWM
- net LCD_BL_PWM: now also R_LCD_BL_GATE.1
- new net LCD_BL: J_LCD_L.8 (Pin_8), J_LCD_R.8 (Pin_8), Q_LCD_BL.3 (D)
- new net LCD_BL_GATE: Q_LCD_BL.1 (G), R_LCD_BL_GATE.2, R_LCD_BL_OFF.2
- no-connect marks 49 -> 48
Other:
- moved on the sheet: C_ADC, C_AMP, C_AMP_BULK, C_BUCK_HF, C_BUCK_IN, C_BUCK_OUT1, C_BUCK_OUT2, C_CAM_AVDD, C_CAM_DVDD, C_CAM_RST, C_EFUSE_DVDT, C_EFUSE_IN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

Commit message: feat(pcb): 新增 J_EXT 调试/外接按键口，并补接线对照表
装进玩偶后板载的 SW_RST / SW_BOOT 按不到。拆解的成品机芯把 3V3/TX/RX/RST/GND
引到板边一排焊盘，这里照做：J_EXT 引出 +3V3 / UART_TX / EN / BOOT / GND。

- 没有 RX：GPIO44（开发板丝印 RX）在本板是舵机 I2C 的 SDA，给不出来。
- BOOT 引出即等于把固件主功能键引出（BOOT_BUTTON_GPIO = GPIO0），外接一个
  按钮同时解决「进下载模式」和「装壳后按不到键」。

选 SH 1.0mm 而不是板上其余连接器统一的 PH 2.0mm：PH 是通孔件，焊盘穿透所有层，
会撞上按键一带 B.Cu 的 LCD_CLK 与 USB_DP（DRC 实测报 shorting_items）；改贴片 PH
后全板扫描只剩一处放得下，且离 EN/BOOT/TX 有 33~48mm。SH 全贴片、8.9x5.3mm，
可贴着两个按键放，引线 3~13mm，对已收敛的布线扰动最小。

同时新增 WIRING.md 接线对照表，由 scripts/export_wiring.py 从 board_spec 生成：
自动测试只能保证 config.h ↔ 原理图 ↔ PCB 内部一致，证明不了「板上器件 = 面包板
实物」，这张表补那个缺口。三个测试防止它与板子脱节。

验证：DRC/未连接/原理图一致性只剩 2 条既有的 U1 丝印告警；116 项测试全过；
fab 与渲染图已重出。

Co-Authored-By: Claude Opus 5 <noreply@anthropic.com>
Parts:
- added J_EXT: Debug / Keys, Connector_JST:JST_SH_BM05B-SRSS-TB_1x05-1MP_P1.00mm_Vertical, symbol Connector_Generic:Conn_01x05
Connections:
- net +3V3: now also J_EXT.1 (Pin_1)
- net BOOT: now also J_EXT.4 (Pin_4)
- net EN: now also J_EXT.3 (Pin_3)
- net GND: now also J_EXT.5 (Pin_5)
- net UART_TX: now also J_EXT.2 (Pin_2)
Other:
- moved on the sheet: C_ADC, C_AMP, C_AMP_BULK, C_BUCK_HF, C_BUCK_IN, C_BUCK_OUT1, C_BUCK_OUT2, C_CAM_AVDD, C_CAM_DVDD, C_CAM_RST, C_EFUSE_DVDT, C_EFUSE_IN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

Commit message: feat(pcb): 麦克风改外接，并把文档与板子实际对齐
板载麦克风要求主板本身放在玩偶能「听见」的位置：塞进胸腔再包一层棉花就废了。
拆解的成品机芯是外接的，改成一样。

- 拆掉 U_MIC / C_MIC / R_MIC_SD，PCB 声孔随 U_MIC 封装一起消失。
- 新增 J_MIC：6 脚 SH 1.0mm 立式座，针序按常见 I2S 麦克风模块丝印
  VDD GND SD WS SCK L/R；末脚给 GND，即 L/R 拉低＝左声道，与原板载
  INMP441 第 4 脚接法一致。兼容 INMP441 / ICS43434 / ZTS6672。
- 座子放在模组右上方而非原麦克风位置：原区域被摄像头扇出线占满，放不下；
  移到 (24.5,18.0) 后三根 MIC 线合计 59.7mm，反而比板载时更短。
- post_route 的声孔避让常量与 remove_microphone_via、fanout 的麦克风地脚
  一并删除，否则整板重新生成时会引用不存在的器件。

ECO 过程中修掉两个脚本缺陷：
- nearest_pad 用 `fp is skip` 跳过座子自身，但 pcbnew 的 SWIG 每次
  GetFootprints() 都返回新代理对象，`is` 永远为假，结果把 J_MIC 自己的焊盘
  当成对端、走线绕回自身。改成按位号比较。
- SH 是 1.0mm 脚距，相邻焊盘只隔 0.4mm，走线从旁边挤不过去（DRC 报
  solder_mask_bridge 与 shorting_items）。每根线先垂直逃出焊盘排再拐弯，
  且逃逸段与 A* 段拼成一条折线一次加入，避免接点对不上。

文档按「以板子实际为准」对齐（委托方 2026-09-15 确认）：
- 摄像头 SCCB 上拉：原写「不贴」，实际 fitted=True，改为「贴」。
- 4.4 节电池预留：原写留 VBAT 焊盘，但 board_spec 从来没有这个网络。改为
  明确不做——单独一个焊盘没用，锂电池要配套升压/充电/保护/电量检测，那是
  一块独立的板子；以后做电池板输出 5V 从 USB-C 或 J_VMOT 进，主板不用改。
- 功放：MAX98357A 或 HT517，板上按 MAX98357A 画，换料前须核封装与针序。

验证：DRC/未连接/原理图一致性只剩 2 条既有的 U1 丝印告警；115 项测试全过；
fab 与渲染图已重出。

Co-Authored-By: Claude Opus 5 <noreply@anthropic.com>
Parts:
- removed C_MIC: 100nF, Capacitor_SMD:C_0402_1005Metric, symbol Device:C
- removed R_MIC_SD: 100k, Resistor_SMD:R_0402_1005Metric, symbol Device:R
- removed U_MIC: INMP441, plush:InvenSense_INMP441_LGA-9_4.72x3.76mm, symbol plush:INMP441
- added J_MIC: Mic, Connector_JST:JST_SH_BM06B-SRSS-TB_1x06-1MP_P1.00mm_Vertical, symbol Connector_Generic:Conn_01x06
Connections:
- net +3V3: now also J_MIC.1 (Pin_1)
- net GND: now also J_MIC.2 (Pin_2), J_MIC.6 (Pin_6)
- net MIC_SCK: now also J_MIC.5 (Pin_5)
- net MIC_SD: now also J_MIC.3 (Pin_3)
- net MIC_WS: now also J_MIC.4 (Pin_4)
Other:
- moved on the sheet: C_AMP, C_AMP_BULK, H1, H2, H3, H4, J_SPK, R_AMP_SD, TP_3V3, TP_GND, TP_PGND, TP_SCL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

Commit message: docs(pcb): 按实有仪器重写首板验收，并补外购件清单
委托方首板只有万用表，没有示波器、限流电源和热像仪；打样贴 5 块。原清单按
齐全仪器写的，照做会得到一堆做不了或做了也证明不了的项。

TESTING.md 重写：
- 新增「仪器与降级」：每个原本要示波器/热像仪的项写明降级做法，并明确列出
  降级后**不能**证明什么——不把「看着正常」当成「验证通过」。
- 新增五块板分工：主力 / 对照 / 牺牲板 / 留存。对照板的用途是回答「这是设计
  问题还是这块焊坏了」，没有它这个问题只能靠猜。
- 新增顺序门禁：逻辑域全通过才接外设，外设全通过才接 VMOT，VMOT 通过才接加热。
  VMOT 那一路没有 eFuse 保护，只能靠顺序兜底。
- 新增接屏前的背光限流检查：J_LCD.8 到 Q_LCD_BL 之间没有限流电阻，当初按
  「屏模块自带」设计但从未验证过。先单眼、先串 100Ω、看电流增量。
- 新增单点接地的测量方法：拆 R_STAR 后量 GND 对 PGND 应开路。
- 用上板上 21 个测试点（原清单一个都没提到）。
- 新增麦克风 L/R 分支：板上 J_MIC 6 脚接 GND 即左声道，静音则改接 3V3。
- 新增「卡住时先查什么」故障表。

WIRING.md 新增外购件清单：屏必须换成 8 针带 BL 版（面包板上的 7 针插不上），
并说明屏线建议用 30AWG 硅胶线而不是杜邦线。

board_spec：J_EXT / J_MIC 由手工件改为贴片件。板上其余手工件都是通孔件，
这两个是 1.0mm 脚距贴片座，手焊容易连锡且 J_MIC 的连锡很隐蔽。
料号 C160391 / C160392；C160391 库存显示不稳定，已在清单里列为下单前确认项。

Co-Authored-By: Claude Opus 5 <noreply@anthropic.com>
Parts:
- J_EXT: LCSC (none) -> C160391; now in the parts list
- J_MIC: LCSC (none) -> C160392; now in the parts list
Changed lines of the file:
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@@
 		(unit 1)
 		(exclude_from_sim no)
-		(in_bom no)
+		(in_bom yes)
 		(on_board yes)
 		(dnp no)
@@
 			)
 		)
+		(property "LCSC" "C160391"
+			(at 513.08 48.26 0)
+			(effects
+				(font
+					(size 1.27 1.27)
+				)
+				(hide yes)
+			)
+		)
 		(pin "1"
 		)
@@
 		(unit 1)
 		(exclude_from_sim no)
-		(in_bom no)
+		(in_bom yes)
 		(on_board yes)
 		(dnp no)
@@
 			(at 990.60 421.64 0)
 			(effects
+				(font
+					(size 1.27 1.27)
+				)
+				(hide yes)
+			)
+		)
+		(property "LCSC" "C160392"
+			(at 990.60 421.64 0)
+			(effects
