File: hardware/plush-toy-mainboard/plush-toy-mainboard.kicad_pcb (KiCad board)
At the start: 4 copper layers, 90 x 60 mm, 115 parts, among them U1 ESP32-S3-WROOM-1-N16R8

Commit message: feat(pcb): regenerate board and fab outputs after review fixes
Board produced by apply_review_eco.py + post_route.py --apply from
c7b9cb5: 0 DRC errors (2 reviewed U1 silk warnings), 0 unconnected,
schematic parity clean; BOM/CPL/Gerber re-exported and validated.

Co-Authored-By: Claude Opus 5 <noreply@anthropic.com>
Claude-Session: https://claude.ai/code/session_01T5KDAGxc5qt48yo4LHintC
Parts:
- turned C_BUCK_IN to 180 degrees
Routing:
- net VBUS: track 98.2 -> 93.7 mm
- net GND: track 149.2 -> 148.5 mm, vias 112 -> 111
Changed lines of the file:
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@@
 	(footprint "Capacitor_SMD:C_0805_2012Metric"
 		(layer "F.Cu")
-		(at 40 11)
+		(at 40 11 180)
 		(descr "Capacitor SMD 0805 (2012 Metric), square (rectangular) end terminal, IPC-7351 nominal, (Body size source: IPC-SM-782 page 76, https://www.pcb-3d.com/wordpress/wp-content/uploads/ipc-sm-782a_amendment_1_and_2.pdf, https://docs.google.com/spreadsheets/d/1BsfQQcO9C6DZCsRaXUlFlo91Tg2WpOkGARC1WS5S8t0/edit?usp=sharing)")
 		(tags "capacitor")
 		(property "Reference" "C_BUCK_IN"
-			(at 0 -1.68 0)
+			(at 0 -1.68 180)
 			(layer "F.SilkS")
 			(hide yes)
@@
 		)
 		(property "Value" "22uF"
-			(at 0 1.68 0)
+			(at 0 1.68 180)
 			(layer "F.Fab")
 			(hide yes)
@@
 		)
 		(property "Datasheet" ""
-			(at 0 0 0)
+			(at 0 0 180)
 			(layer "F.Fab")
 			(hide yes)
@@
 		)
 		(property "Description" ""
-			(at 0 0 0)
+			(at 0 0 180)
 			(layer "F.Fab")
 			(hide yes)
@@
 		)
 		(property "KiLib_Generator" "SMD_2terminal_chip_molded"
-			(at 0 0 0)
+			(at 0 0 180)
 			(layer "F.SilkS")
 			(hide yes)
@@
 		)
 		(property "LCSC" "C45783"
-			(at 0 0 0)
+			(at 0 0 180)
 			(layer "F.SilkS")
 			(hide yes)
@@
 		(duplicate_pad_numbers_are_jumpers no)
 		(fp_line
-			(start -0.261252 -0.735)
-			(end 0.261252 -0.735)
+			(start -0.261252 0.735)
+			(end 0.261252 0.735)
 			(stroke
 				(width 0.12)
@@
 		)
 		(fp_line
-			(start -0.261252 0.735)
-			(end 0.261252 0.735)
+			(start -0.261252 -0.735)
+			(end 0.261252 -0.735)
 			(stroke
 				(width 0.12)
@@
 		)
 		(fp_text user "${REFERENCE}"
-			(at 0 0 0)
+			(at 0 0 180)
 			(layer "F.Fab")
 			(effects
@@
 		)
 		(pad "1" smd roundrect
-			(at -0.95 0)
+			(at -0.95 0 180)
 			(size 1 1.45)
 			(layers "F.Cu" "F.Mask" "F.Paste")
@@
 		)
 		(pad "2" smd roundrect
-			(at 0.95 0)
+			(at 0.95 0 180)
 			(size 1 1.45)
 			(layers "F.Cu" "F.Mask" "F.Paste")
@@
 		(at 70.5 14.8)
 		(property "Reference" "C_VMOT_BULK"
-			(at -8.295001 -0.000001 90)
+			(at 0 -7.795 0)
 			(layer "F.SilkS")
 			(effects
@@
 		(tags "mountinghole M3")
 		(property "Reference" "H3"
-			(at -5.79247 0 0)
+			(at 0.001264 5.097526 0)
 			(layer "F.SilkS")
 			(effects
@@
 		(layer "Edge.Cuts")
 	)
-	(gr_text "头部触摸 E0 / GND"
-		(at 10 45 0)
+	(gr_text "头部触摸\nE0 / GND"
+		(at 11.6 56 0)
 		(layer "F.SilkS")
 		(effects
@@
 		)
 	)
-	(gr_text "电机/加热专用 5V"
-		(at 70 7 0)
+	(gr_text "必须串 KSD9700 65度 常闭"
+		(at 70 39.6 0)
 		(layer "F.SilkS")
 		(effects
@@
 		)
 	)
-	(gr_text "必须串 KSD9700 65度 常闭"
-		(at 70 39.6 0)
+	(gr_text "CH0 左"
+		(at 73.5 28 0)
 		(layer "F.SilkS")
 		(effects
@@
 		)
 	)
-	(gr_text "VMOT 仅限 5V"
-		(at 70.5 2.999999 0)
+	(gr_text "-"
+		(at 80.8 11.42 0)
 		(layer "F.SilkS")
 		(effects
@@
 		)
 	)
-	(gr_text "CH0 左"
-		(at 73.5 28 0)
+	(gr_text "+"
+		(at 80.8 16.5 0)
 		(layer "F.SilkS")
 		(effects
@@
 		)
 	)
-	(gr_text "-"
-		(at 80.8 11.42 0)
+	(gr_text "CH1 右"
+		(at 81 32 0)
 		(layer "F.SilkS")
 		(effects
@@
 		)
 	)
-	(gr_text "+"
-		(at 80.8 16.5 0)
+	(gr_text "VMOT 仅限 5V"
+		(at 83.899999 3.099999 0)
 		(layer "F.SilkS")
 		(effects
@@
 				(thickness 0.15)
 			)
+			(justify right)
 		)
 	)
-	(gr_text "CH1 右"
-		(at 81 32 0)
+	(gr_text "电机/加热专用 5V"
+		(at 83.899999 5 0)
 		(layer "F.SilkS")
 		(effects
@@
 				(thickness 0.15)
 			)
+			(justify right)
 		)
 	)
@@
 	)
 	(segment
+		(start 39.05 11)
+		(end 39.1 11)
+		(width 0.4)
+		(layer "F.Cu")
+		(net "GND")
+	)
+	(segment
 		(start 32.3154 9.2817)
 		(end 32.1143 9.0806)
@@
 	)
 	(segment
-		(start 40.95 11)
-		(end 41 11.75)
-		(width 0.4)
-		(layer "F.Cu")
-		(net "GND")
-	)
-	(segment
 		(start 11.08 40.85)
 		(end 18.8 40.85)
@@
 	)
 	(via
-		(at 40.95 11)
-		(size 0.6)
-		(drill 0.3)
-		(layers "F.Cu" "B.Cu")
-		(net "GND")
-	)
-	(via
 		(at 31.52 50.15)
 		(size 0.6)
@@
 	)
 	(via
-		(at 41 11.75)
-		(size 0.6)
-		(drill 0.3)
-		(layers "F.Cu" "B.Cu")
-		(net "GND")
-	)
-	(via
 		(at 18.8 42.15)
 		(size 0.6)
@@
 	)
 	(via
+		(at 39.1 11)
+		(size 0.6)
+		(drill 0.3)
+		(layers "F.Cu" "B.Cu")
+		(net "GND")
+	)
+	(via
 		(at 58.5602 30.6771)
 		(size 0.6)
@@
 	)
 	(segment
-		(start 35 3.35)
-		(end 33.8564 4.4936)
-		(width 0.2)
+		(start 33.6 11.1)
+		(end 33.6 11.3)
+		(width 0.5)
+		(locked yes)
 		(layer "F.Cu")
 		(net "VBUS_FUSED")
 	)
 	(segment
-		(start 33.8564 11.2753)
-		(end 34 11.3)
+		(start 33.549999 18.75)
+		(end 33.549999 19.25)
 		(width 0.2)
 		(layer "F.Cu")
@@
 	)
 	(segment
-		(start 34 5.1)
-		(end 33.7 5.1)
+		(start 33.3 11.4)
+		(end 33.3 11.5)
 		(width 0.5)
+		(locked yes)
 		(layer "F.Cu")
 		(net "VBUS_FUSED")
 	)
 	(segment
-		(start 34 4.5)
-		(end 34 5.1)
+		(start 33.5 11.3)
+		(end 33.5 11.4)
 		(width 0.5)
+		(locked yes)
 		(layer "F.Cu")
 		(net "VBUS_FUSED")
 	)
 	(segment
-		(start 32.8 12.2)
-		(end 32.8 18.4)
+		(start 33.7 3.4)
+		(end 33.7 11.1)
 		(width 0.5)
+		(locked yes)
 		(layer "F.Cu")
 		(net "VBUS_FUSED")
 	)
 	(segment
-		(start 33.7 11.3)
-		(end 34 11.3)
+		(start 33.549999 19.25)
+		(end 31.48 19.25)
 		(width 0.5)
 		(layer "F.Cu")
@@
 	)
 	(segment
-		(start 33 12.2)
-		(end 32.8 12.2)
+		(start 33.3 11.5)
+		(end 32.5 11.5)
 		(width 0.5)
+		(locked yes)
 		(layer "F.Cu")
 		(net "VBUS_FUSED")
 	)
 	(segment
-		(start 33.253 18.75)
-		(end 33.55 18.75)
-		(width 0.2)
-		(layer "F.Cu")
-		(net "VBUS_FUSED")
-	)
-	(segment
-		(start 33.7 5.1)
-		(end 33.7 11.3)
+		(start 34.9 3.4)
+		(end 33.7 3.4)
 		(width 0.5)
+		(locked yes)
 		(layer "F.Cu")
 		(net "VBUS_FUSED")
 	)
 	(segment
-		(start 33.55 18.75)
-		(end 33.55 19.75)
-		(width 0.2)
-		(layer "F.Cu")
-		(net "VBUS_FUSED")
-	)
-	(segment
-		(start 32.9351 12.1966)
-		(end 33 12.2)
+		(start 33.549999 19.25)
+		(end 33.549999 19.75)
 		(width 0.2)
 		(layer "F.Cu")
@@
 	)
 	(segment
-		(start 32.9351 18.4321)
-		(end 32.8 18.4)
-		(width 0.2)
+		(start 32.5 11.5)
+		(end 32.5 19.25)
+		(width 0.5)
+		(locked yes)
 		(layer "F.Cu")
 		(net "VBUS_FUSED")
 	)
 	(segment
-		(start 33.8564 11.2753)
-		(end 32.9351 12.1966)
-		(width 0.2)
+		(start 33.6 11.3)
+		(end 33.5 11.3)
+		(width 0.5)
+		(locked yes)
 		(layer "F.Cu")
 		(net "VBUS_FUSED")
 	)
 	(segment
-		(start 33.8564 4.4936)
-		(end 34 4.5)
-		(width 0.2)
+		(start 33.7 11.1)
+		(end 33.6 11.1)
+		(width 0.5)
+		(locked yes)
 		(layer "F.Cu")
 		(net "VBUS_FUSED")
 	)
 	(segment
-		(start 32.9351 18.4321)
-		(end 33.253 18.75)
-		(width 0.2)
+		(start 35 3.35)
+		(end 34.9 3.4)
+		(width 0.5)
+		(locked yes)
 		(layer "F.Cu")
 		(net "VBUS_FUSED")
 	)
 	(segment
-		(start 33.55 19.25)
-		(end 31.48 19.25)
+		(start 33.5 11.4)
+		(end 33.3 11.4)
 		(width 0.5)
+		(locked yes)
 		(layer "F.Cu")
 		(net "VBUS_FUSED")
@@
 	)
 	(segment
-		(start 40 11)
-		(end 39.05 11)
-		(width 0.5)
-		(layer "F.Cu")
-		(net "VBUS")
-	)
-	(segment
 		(start 28.75 20.6776)
 		(end 31.5402 23.4678)
@@
 	)
 	(segment
+		(start 42.25 11)
+		(end 40.95 11)
+		(width 0.5)
+		(layer "F.Cu")
+		(net "VBUS")
+	)
+	(segment
 		(start 39.68 16.49)
 		(end 40.4173 16.49)
@@
 	)
 	(segment
-		(start 42.25 9.7)
-		(end 40 9.7)
-		(width 0.5)
-		(layer "F.Cu")
-		(net "VBUS")
-	)
-	(segment
 		(start 36.5 19.75)
 		(end 39.26 19.75)
@@
 	)
 	(segment
-		(start 42.25 14.95)
-		(end 42.25 9.7)
-		(width 0.5)
-		(layer "F.Cu")
-		(net "VBUS")
-	)
-	(segment
 		(start 55.2088 54.015)
 		(end 55.375 54.015)
@@
 	)
 	(segment
+		(start 42.25 14.95)
+		(end 42.25 11)
+		(width 0.5)
+		(layer "F.Cu")
+		(net "VBUS")
+	)
+	(segment
 		(start 35.45 19.7771)
 		(end 35.45 19.75)
@@
 		(width 0.5)
 		(layer "F.Cu")
-		(net "VBUS")
-	)
-	(segment
-		(start 40 9.7)
-		(end 40 11)
-		(width 0.5)
-		(layer "F.Cu")

Commit message: feat(pcb): GPIO48 改驱动双眼背光，撤销板载 RGB 灯
屏幕换成带独立 BL 引脚的型号（7 针 → 8 针 RST/CS/DC/SDA/SCL/GND/VCC/BL）。
D_LED 与 C_LED 整体撤销，GPIO48 改作两眼共用的 25kHz 背光 PWM：眼睛本身已能
表达设备状态，换来统一亮度调节和休眠关背光。摄像头、音频、USB、SPI 与
strapping 脚均不受影响。

硬件：
- 新增 AO3401A 高边开关 Q_LCD_BL（与 Q_REV 同料号 C15127），栅极串 100Ω、
  上拉 100k 至 +3V3，保证 LEDC 配置前 GPIO48 浮空时背光默认灭。
- 开关放在双屏排针正下方的空区：LCD_BL 只需 4~11mm 就接到两排 8 脚，横穿
  板子的改成 25kHz 栅极信号。此处 x<62，In2.Cu 的 +3V3 覆铜仍在（覆铜止于
  x=62），源极和上拉能就近打孔取电。
- 新增 apply_backlight_eco.py：整板重新自动布线会在 U_TOUCH/J_CAM 密集区失去
  已收敛路径，因此只做局部 ECO，且 DRC/未连接/原理图一致性全过才覆盖正式 PCB。
- 排针加到 8 针后 8 脚右移 2.54mm，J_VMOT 旁两行 5V 警告标签离屏排针只剩
  5.5mm，又会被读成「屏幕座是 5V」——正是 2026-09-14 评审要消除的误读。右边
  顶着 H3 安装孔挪不动，故第二行去掉与第一行重复的「5V」，只留设计方案要求的
  「电机/加热专用」，两行右挪后间距 7.4mm。

固件：
- DISPLAY_BACKLIGHT_PIN=GPIO48 + DISPLAY_BACKLIGHT_OUTPUT_INVERT（低电平导通
  高边 P-MOS），改用 PwmBacklight；移除 GetLed 覆写，回落到基类 NoLed。

验证：DRC/未连接/原理图一致性只剩 2 条既有的 U1 丝印告警；113 项测试全过；
idf.py build 通过；fab 与渲染图已重出。

Co-Authored-By: Claude Opus 5 <noreply@anthropic.com>
Parts:
- removed C_LED: 100nF, Capacitor_SMD:C_0402_1005Metric
- removed D_LED: WS2812B-2020-V6, LED_SMD:LED_WS2812B-2020_PLCC4_2.0x2.0mm
- removed the J_LCD_L at (47.0, 2.50)
- removed the J_LCD_R at (47.0, 7.50)
- added J_LCD_L: LCD L, Connector_PinHeader_2.54mm:PinHeader_1x08_P2.54mm_Vertical, F.Cu at (47.0, 2.50)
- added J_LCD_R: LCD R, Connector_PinHeader_2.54mm:PinHeader_1x08_P2.54mm_Vertical, F.Cu at (47.0, 7.50)
- added Q_LCD_BL: AO3401A, Package_TO_SOT_SMD:SOT-23, F.Cu at (60.0, 13.0)
- added R_LCD_BL_GATE: 100, Resistor_SMD:R_0402_1005Metric, F.Cu at (56.8, 12.1)
- added R_LCD_BL_OFF: 100k, Resistor_SMD:R_0402_1005Metric, F.Cu at (57.0, 10.3)
Connections:
- U1 pad 25: LED_RGB -> LCD_BL_PWM
Routing:
- net LCD_BL_PWM: track 0.00 -> 53.2 mm, vias 0 -> 2
- net LCD_BL: track 0.00 -> 14.4 mm
- net LED_RGB: track 11.6 -> 0.00 mm, vias 2 -> 0
- net LCD_BL_GATE: track 0.00 -> 5.06 mm
- net GND: track 148.5 -> 146.9 mm, vias 111 -> 109
- net +3V3: track 71.6 -> 70.2 mm
Other:
- board text added: "电机/加热专用"
- board text removed: "电机/加热专用 5V"

Commit message: feat(pcb): 新增 J_EXT 调试/外接按键口，并补接线对照表
装进玩偶后板载的 SW_RST / SW_BOOT 按不到。拆解的成品机芯把 3V3/TX/RX/RST/GND
引到板边一排焊盘，这里照做：J_EXT 引出 +3V3 / UART_TX / EN / BOOT / GND。

- 没有 RX：GPIO44（开发板丝印 RX）在本板是舵机 I2C 的 SDA，给不出来。
- BOOT 引出即等于把固件主功能键引出（BOOT_BUTTON_GPIO = GPIO0），外接一个
  按钮同时解决「进下载模式」和「装壳后按不到键」。

选 SH 1.0mm 而不是板上其余连接器统一的 PH 2.0mm：PH 是通孔件，焊盘穿透所有层，
会撞上按键一带 B.Cu 的 LCD_CLK 与 USB_DP（DRC 实测报 shorting_items）；改贴片 PH
后全板扫描只剩一处放得下，且离 EN/BOOT/TX 有 33~48mm。SH 全贴片、8.9x5.3mm，
可贴着两个按键放，引线 3~13mm，对已收敛的布线扰动最小。

同时新增 WIRING.md 接线对照表，由 scripts/export_wiring.py 从 board_spec 生成：
自动测试只能保证 config.h ↔ 原理图 ↔ PCB 内部一致，证明不了「板上器件 = 面包板
实物」，这张表补那个缺口。三个测试防止它与板子脱节。

验证：DRC/未连接/原理图一致性只剩 2 条既有的 U1 丝印告警；116 项测试全过；
fab 与渲染图已重出。

Co-Authored-By: Claude Opus 5 <noreply@anthropic.com>
Parts:
- added J_EXT: Debug / Keys, Connector_JST:JST_SH_BM05B-SRSS-TB_1x05-1MP_P1.00mm_Vertical, F.Cu at (17.8, 9.75)
Routing:
- net UART_TX: track 29.8 -> 54.6 mm
- net EN: track 49.8 -> 59.5 mm
- net BOOT: track 18.4 -> 24.9 mm, vias 0 -> 2
- net GND: track 146.9 -> 147.0 mm, vias 109 -> 110
- net +3V3: track 70.2 -> 70.3 mm, vias 34 -> 35

Commit message: feat(pcb): 麦克风改外接，并把文档与板子实际对齐
板载麦克风要求主板本身放在玩偶能「听见」的位置：塞进胸腔再包一层棉花就废了。
拆解的成品机芯是外接的，改成一样。

- 拆掉 U_MIC / C_MIC / R_MIC_SD，PCB 声孔随 U_MIC 封装一起消失。
- 新增 J_MIC：6 脚 SH 1.0mm 立式座，针序按常见 I2S 麦克风模块丝印
  VDD GND SD WS SCK L/R；末脚给 GND，即 L/R 拉低＝左声道，与原板载
  INMP441 第 4 脚接法一致。兼容 INMP441 / ICS43434 / ZTS6672。
- 座子放在模组右上方而非原麦克风位置：原区域被摄像头扇出线占满，放不下；
  移到 (24.5,18.0) 后三根 MIC 线合计 59.7mm，反而比板载时更短。
- post_route 的声孔避让常量与 remove_microphone_via、fanout 的麦克风地脚
  一并删除，否则整板重新生成时会引用不存在的器件。

ECO 过程中修掉两个脚本缺陷：
- nearest_pad 用 `fp is skip` 跳过座子自身，但 pcbnew 的 SWIG 每次
  GetFootprints() 都返回新代理对象，`is` 永远为假，结果把 J_MIC 自己的焊盘
  当成对端、走线绕回自身。改成按位号比较。
- SH 是 1.0mm 脚距，相邻焊盘只隔 0.4mm，走线从旁边挤不过去（DRC 报
  solder_mask_bridge 与 shorting_items）。每根线先垂直逃出焊盘排再拐弯，
  且逃逸段与 A* 段拼成一条折线一次加入，避免接点对不上。

文档按「以板子实际为准」对齐（委托方 2026-09-15 确认）：
- 摄像头 SCCB 上拉：原写「不贴」，实际 fitted=True，改为「贴」。
- 4.4 节电池预留：原写留 VBAT 焊盘，但 board_spec 从来没有这个网络。改为
  明确不做——单独一个焊盘没用，锂电池要配套升压/充电/保护/电量检测，那是
  一块独立的板子；以后做电池板输出 5V 从 USB-C 或 J_VMOT 进，主板不用改。
- 功放：MAX98357A 或 HT517，板上按 MAX98357A 画，换料前须核封装与针序。

验证：DRC/未连接/原理图一致性只剩 2 条既有的 U1 丝印告警；115 项测试全过；
fab 与渲染图已重出。

Co-Authored-By: Claude Opus 5 <noreply@anthropic.com>
Parts:
- removed C_MIC: 100nF, Capacitor_SMD:C_0402_1005Metric
- removed R_MIC_SD: 100k, Resistor_SMD:R_0402_1005Metric
- removed U_MIC: INMP441, plush:InvenSense_INMP441_LGA-9_4.72x3.76mm
- added J_MIC: Mic, Connector_JST:JST_SH_BM06B-SRSS-TB_1x06-1MP_P1.00mm_Vertical, F.Cu at (24.5, 18.0)
Routing:
- net MIC_SD: track 39.8 -> 27.6 mm, vias 2 -> 4
- net MIC_WS: track 37.9 -> 29.9 mm, vias 2 -> 6
- net MIC_SCK: track 35.0 -> 29.7 mm, vias 2 -> 6
- net +3V3: track 70.3 -> 69.6 mm, vias 35 -> 33
- net GND: track 147.0 -> 146.7 mm, vias 110 -> 106
